File: Pollen PCB/Pollen PCB.kicad_pcb (KiCad board)
At the start: 2 copper layers, 115.5 x 82.2 mm, 30 parts, among them J1 GY-GPS6MV2, J2 Adafruit Charge Controller, J3 Solar_panel, J4 Solar_panel, J5 Solar_charger, J6 Raspberry Pi, J7 Battery, J8 RPi power, Q1 Si2319CDS, Q2 MMBT2222A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

Commit message: Generate fab files
Parts:
- moved C1 264.6 mm to (-90.0, -47.0)
- moved J1 264.6 mm to (-56.4, -39.0)
- moved J2 264.6 mm to (-107.8, -44.8)
- moved J3 264.6 mm to (-87.5, -74.8)
- moved J4 264.6 mm to (-91.5, -74.8)
- moved J5 264.6 mm to (-95.5, -74.8)
- moved J6 264.6 mm to (-3.98, -29.6)
- moved J7 264.6 mm to (-99.5, -74.8)
- moved J8 264.6 mm to (-77.5, -36.5)
- moved Q1 264.6 mm to (-79.5, -71.5)
- moved Q2 264.6 mm to (-77.5, -67.2)
- moved Q3 264.6 mm to (-20.8, -32.8)
- moved Q4 264.6 mm to (-19.8, -28.8)
- moved R1 264.6 mm to (-90.5, -67.0)
- moved R10 264.6 mm to (-64.0, -34.5)
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